Commit message: Making arms

File: src/chatboat_description/urdf/chatboat_uvms.urdf.xacro (robot description, xacro)
@@ -1,9 +1,9 @@
 <?xml version="1.0"?>
 <robot xmlns:xacro="http://www.ros.org/wiki/xacro" name="chatboat_uvms">
-  <!-- Composite UVMS: GIRONA500 + ECA 5E + Gripper -->
-  <xacro:include filename="$(find chatboat_description)/urdf/girona500.urdf.xacro"/>
-  <xacro:include filename="$(find chatboat_description)/urdf/eca5e.urdf.xacro"/>
+  <!-- Composite UVMS: BlueROV2 Heavy + Reach Alpha 5 + Gripper -->
+  <xacro:include filename="$(find chatboat_description)/urdf/bluerov2.urdf.xacro"/>
+  <xacro:include filename="$(find chatboat_description)/urdf/alpha5.urdf.xacro"/>
   <xacro:include filename="$(find chatboat_description)/urdf/gripper.urdf.xacro"/>
-  <xacro:arg name="namespace" default="girona500"/>
+  <xacro:arg name="namespace" default="chatboat"/>
   <!-- World frame (NED) -->
   <link name="world"/>
@@ -13,8 +13,8 @@
   </joint>
   <!-- Instantiate vehicle -->
-  <xacro:girona500 namespace="$(arg namespace)"/>
-  <!-- Instantiate arm (mounted at front-bottom of vehicle) -->
-  <xacro:eca5e parent="$(arg namespace)/base_link" namespace="$(arg namespace)"/>
+  <xacro:bluerov2 namespace="$(arg namespace)"/>
+  <!-- Instantiate arm (mounted at front of vehicle) -->
+  <xacro:alpha5 parent="$(arg namespace)/base_link" namespace="$(arg namespace)"/>
   <!-- Instantiate gripper (at end of arm) -->
-  <xacro:gripper parent="arm_link4"/>
+  <xacro:gripper parent="arm_wrist"/>
 </robot>

File: src/chatboat_description/urdf/gripper.urdf.xacro (robot description, xacro)
@@ -29,5 +29,5 @@
       <parent link="${parent}"/>
       <child link="gripper_tip"/>
-      <origin xyz="0.10 0 0" rpy="0 0 0"/>
+      <origin xyz="0 0 0.14" rpy="0 0 0"/>
     </joint>
     <!-- End-effector frame (control reference point) -->
