Commit message: Robotic arm fix?

File: src/chatboat_description/urdf/alpha5.urdf.xacro (robot description, xacro)
@@ -105,4 +105,20 @@
       <limit lower="0.0" upper="3.22" effort="9.0" velocity="0.5"/>
     </joint>
+    <link name="arm_tcp_adapter">
+      <visual>
+        <geometry><cylinder radius="0.020" length="0.040"/></geometry>
+        <origin xyz="0 0 0.02"/>
+        <material name="arm_dark"/>
+      </visual>
+      <inertial><mass value="0.050"/>
+        <origin xyz="0 0 0.02"/>
+        <inertia ixx="0.00001" ixy="0" ixz="0" iyy="0.00001" iyz="0" izz="0.00001"/>
+      </inertial>
+    </link>
+    <joint name="tcp_adapter_joint" type="fixed">
+      <parent link="arm_wrist"/>
+      <child link="arm_tcp_adapter"/>
+      <origin xyz="0 0 0.09975"/>
+    </joint>
   </xacro:macro>
 </robot>

File: src/chatboat_description/urdf/chatboat_uvms.urdf.xacro (robot description, xacro)
@@ -17,4 +17,4 @@
   <xacro:alpha5 parent="$(arg namespace)/base_link" namespace="$(arg namespace)"/>
   <!-- Instantiate gripper (at end of arm) -->
-  <xacro:gripper parent="arm_wrist"/>
+  <xacro:gripper parent="arm_tcp_adapter"/>
 </robot>

File: src/chatboat_description/urdf/gripper.urdf.xacro (robot description, xacro)
@@ -29,5 +29,5 @@
       <parent link="${parent}"/>
       <child link="gripper_tip"/>
-      <origin xyz="0 0 0.14" rpy="0 0 0"/>
+      <origin xyz="0 0 0.04" rpy="0 0 0"/>
     </joint>
     <!-- End-effector frame (control reference point) -->
